File: Buck/Buck.kicad_pcb (KiCad board)
At the start: 2 copper layers, 260 x 190 mm, 22 parts, among them Q2 IRFZ44, U1 HCPL-3180

Commit message: [SAVED]
Parts:
- moved Vin-GeradorSinal1 1.00 mm to (99.0, 59.0)
Changed lines of the file:
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@@
 	(footprint "Buck:SMD50"
 		(layer "F.Cu")
-		(at 98 59)
+		(at 99 59)
 		(property "Reference" "Vin-GeradorSinal1"
 			(at 1.54 -7.67 0)
